File: PCBs/PhotonPowerZeroSchematic_Informational_Only.kicad_sch (KiCad schematic)
At the start: 27 parts, among them J1 Raspberry_Pi_2_3, U1 TPS613222ADBV, U2 AP2161W, U3 BQ24074RGT, U4 MCP1700x-330xxMB, U5 ATtiny84A-SS

Commit message: Schematic Udate
Parts:
- added R10, R11, R12, R9: 1k, symbol Device:R
Connections:
- net VCC: now also R11.2, R12.2; no longer D2.1 (K), D3.1 (K)
- net at U5.6 (PA7): now also R10.1; no longer D4.2 (A)
- net at U5.7 (PA6): now also R9.1; no longer D5.2 (A)
- new net: D4.2 (A), R10.2
- new net: D2.1 (K), R11.1
- new net: D5.2 (A), R9.2
- new net: D3.1 (K), R12.1

Commit message: minor pcb and schematic updates!
Connections:
- net GND: now also C1.2; no longer C1.1
- net at D1.1 (K), J1.2 (5V), U1.4 (VOUT): now also C1.1; no longer C1.2
Other:
- moved on the sheet: C1, C6, R2
