File: PCBs/Photon_Power_Zero_PCB_r1_02.kicad_pcb (KiCad board)
At the start: 2 copper layers, 65.1 x 30.1 mm, 56 parts, among them J1 JST_S2B-PH-SM4-TB_LF__SN_, J2 JST_GH_SM02B-GHS-TB_1x02-1MP_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, J3 SMT_Solar_barrel, U1 ATtiny84-SSFR, U2 REG_MCP1700T-3602E/MB, U3 bq2407, U4 AP2161-WG, U5 TPS613222A

Commit message: changes for rev2 and cleanup
Parts:
- added G***: LOGO, LOGO, B.Cu at (179.0, 91.8)
- added REF**: PinHeader_1x02_P2.54mm_Vertical, Pin headers:PinHeader_1x02_P2.54mm_Vertical, F.Cu at (194.7, 81.2)
- moved FID4 0.66 mm to (193.8, 78.2)
Routing:
- net VccSolar: track 46.9 -> 60.3 mm
- net GND: track 71.6 -> 79.1 mm
Other:
- board text added: "+ -"
- board text added: "CERN Open Hardware Licence V2(CERN-OHL-S)"
- board text added: "Li-Ion (3.7v)"
- board text added: "MAX 12V"
- board text added: "Photon Power Zero"
- board text removed: "3.7V"
- board text removed: "CERN Open Hardware Licence V2"
- board text removed: "CERN-OHL-S"
- board text removed: "Li-Ion"
- board text removed: "MAX 9V"

Commit message: update
Parts:
- removed the G*** at (152.0, 99.5)
- removed the G*** at (179.0, 91.8)
- added G***: LOGO, LOGO, F.Cu at (174.2, 87.6)
