File: PCBs/experimental/RFM69HCW_v6.kicad_pcb (KiCad board)
At the start: 2 copper layers, 65.1 x 30.1 mm, 12 parts

Commit message: PCB rev
Parts:
- moved D1 1.70 mm to (139.1, 98.3), turned to -90 degrees
- moved REF** 0.16 mm to (135.8, 89.3)
Connections:
- REF** pad DIO0: INTER -> INTER433
- REF** pad 03: (no net) -> 5v2RPi
- REF** pad 3v3: 3v3 -> (no net)
- REF** pad DIO0: INTER -> INTER915
Routing:
- net INTER: track 66.5 -> 0.00 mm, vias 4 -> 0
- net INTER915: track 0.00 -> 39.2 mm, vias 0 -> 2
- net INTER433: track 0.00 -> 29.1 mm, vias 0 -> 2
- net 3v3: track 79.5 -> 66.3 mm, vias 0 -> 3
- net MOSI: track 39.2 -> 29.7 mm, vias 4 -> 2
- net MISO: track 36.5 -> 28.4 mm, vias 2 -> 3
- net SLCK: track 31.2 -> 26.7 mm
- net CS1: track 22.1 -> 19.1 mm
- net RST: track 35.0 -> 33.3 mm
- net GND: vias 118 -> 137
- added copper zone on In1.Cu, net 3v3
- added copper zone on In2.Cu, net 3v3
Other:
- copper layers 2 -> 4
